Commit message: Added a forklift section

File: install/TeleARM/share/TeleARM/urdf/telearm.urdf.xacro (robot description, xacro)
@@ -119,4 +119,11 @@
     </visual>
   </link>
+  <link name = "fork_lift_link" type = "prismatic">
+    <visual>
+      <geometry>
+        <box size="0.4 0.15 0.05"/>
+      </geometry>
+    </visual>
+  </link>
   <joint name="body_to_window" type="fixed">
     <origin xyz="0 0 0"/>
@@ -147,4 +154,11 @@
     <child link="back_right_wheel"/>
     <axis xyz="0 0 -1"/>
+  </joint>
+  <joint name = "body_to_fork_lift_link" type = "prismatic">
+    <origin xyz="0 0 0" rpy="0 0 0"/>
+    <parent link="body"/>
+    <child link="fork_lift_link"/>
+    <axis xyz="0 0 1"/>
+    <limit effort="50" velocity="0.2" lower="0" upper="0.5"/>
   </joint>
   <link name="lidar_link"/>

Commit message: Added ForkPlate

File: install/TeleARM/share/TeleARM/urdf/telearm.urdf.xacro (robot description, xacro)
@@ -119,9 +119,17 @@
     </visual>
   </link>
-  <link name = "fork_lift_link" type = "prismatic">
-    <visual>
-      <geometry>
-        <box size="0.4 0.15 0.05"/>
-      </geometry>
+  <link name="fork_lift_link">
+    <inertial>
+      <mass value="0.5"/>
+      <inertia ixx="0.01" ixy="0" ixz="0" iyy="0.01" iyz="0" izz="0.01"/>
+    </inertial>
+    <visual>
+      <origin xyz="0 0 0" rpy="0 0 0"/>
+      <geometry>
+        <box size="1.25 1.50 0.08"/>
+      </geometry>
+      <material name="green">
+        <color rgba="0 1 0 1"/>
+      </material>
     </visual>
   </link>
@@ -155,10 +163,10 @@
     <axis xyz="0 0 -1"/>
   </joint>
-  <joint name = "body_to_fork_lift_link" type = "prismatic">
-    <origin xyz="0 0 0" rpy="0 0 0"/>
+  <joint name="body_to_fork_lift_link" type="prismatic">
+    <origin xyz="2.6 0 0.10" rpy="0 0 0"/>
     <parent link="body"/>
     <child link="fork_lift_link"/>
     <axis xyz="0 0 1"/>
-    <limit effort="50" velocity="0.2" lower="0" upper="0.5"/>
+    <limit effort="50" velocity="0.2" lower="-0.10" upper="0.419"/>
   </joint>
   <link name="lidar_link"/>

Commit message: Added Gripper

File: install/TeleARM/share/TeleARM/urdf/telearm.urdf.xacro (robot description, xacro)
@@ -119,7 +119,8 @@
     </visual>
   </link>
-  <link name="fork_lift_link">
-    <inertial>
-      <mass value="0.5"/>
+  <!-- Simple underbody gripper: base + 2 fingers -->
+  <link name="gripper_base">
+    <inertial>
+      <mass value="0.3"/>
       <inertia ixx="0.01" ixy="0" ixz="0" iyy="0.01" iyz="0" izz="0.01"/>
     </inertial>
@@ -127,8 +128,38 @@
       <origin xyz="0 0 0" rpy="0 0 0"/>
       <geometry>
-        <box size="1.25 1.50 0.08"/>
-      </geometry>
-      <material name="green">
-        <color rgba="0 1 0 1"/>
+        <box size="0.25 0.35 0.05"/>
+      </geometry>
+      <material name="grey">
+        <color rgba="0.4 0.4 0.4 1"/>
+      </material>
+    </visual>
+  </link>
+  <link name="left_finger">
+    <inertial>
+      <mass value="0.1"/>
+      <inertia ixx="0.001" ixy="0" ixz="0" iyy="0.001" iyz="0" izz="0.001"/>
+    </inertial>
+    <visual>
+      <origin xyz="0.15 0 0" rpy="0 0 0"/>
+      <geometry>
+        <box size="0.30 0.04 0.08"/>
+      </geometry>
+      <material name="yellow">
+        <color rgba="1 0.85 0 1"/>
+      </material>
+    </visual>
+  </link>
+  <link name="right_finger">
+    <inertial>
+      <mass value="0.1"/>
+      <inertia ixx="0.001" ixy="0" ixz="0" iyy="0.001" iyz="0" izz="0.001"/>
+    </inertial>
+    <visual>
+      <origin xyz="0.15 0 0" rpy="0 0 0"/>
+      <geometry>
+        <box size="0.30 0.04 0.08"/>
+      </geometry>
+      <material name="yellow">
+        <color rgba="1 0.85 0 1"/>
       </material>
     </visual>
@@ -163,10 +194,23 @@
     <axis xyz="0 0 -1"/>
   </joint>
-  <joint name="body_to_fork_lift_link" type="prismatic">
-    <origin xyz="2.6 0 0.10" rpy="0 0 0"/>
-    <parent link="body"/>
-    <child link="fork_lift_link"/>
-    <axis xyz="0 0 1"/>
-    <limit effort="50" velocity="0.2" lower="-0.10" upper="0.419"/>
+  <!-- Gripper mounts under the front; slide fingers on Y to open/close -->
+  <joint name="body_to_gripper_base" type="fixed">
+    <origin xyz="2.4 0 0.15" rpy="0 0 0"/>
+    <parent link="body"/>
+    <child link="gripper_base"/>
+  </joint>
+  <joint name="gripper_left" type="prismatic">
+    <origin xyz="0 0.08 0" rpy="0 0 0"/>
+    <parent link="gripper_base"/>
+    <child link="left_finger"/>
+    <axis xyz="0 1 0"/>
+    <limit effort="20" velocity="0.2" lower="0.0" upper="0.12"/>
+  </joint>
+  <joint name="gripper_right" type="prismatic">
+    <origin xyz="0 -0.08 0" rpy="0 0 0"/>
+    <parent link="gripper_base"/>
+    <child link="right_finger"/>
+    <axis xyz="0 -1 0"/>
+    <limit effort="20" velocity="0.2" lower="0.0" upper="0.12"/>
   </joint>
   <link name="lidar_link"/>

Commit message: fixed dimmensions of forklift

File: install/TeleARM/share/TeleARM/urdf/telearm.urdf.xacro (robot description, xacro)
@@ -128,8 +128,8 @@
       <origin xyz="0 0 0" rpy="0 0 0"/>
       <geometry>
-        <box size="0.25 0.35 0.05"/>
-      </geometry>
-      <material name="grey">
-        <color rgba="0.4 0.4 0.4 1"/>
+        <box size="0.5 1.0 0.05"/>
+      </geometry>
+      <material name="green">
+        <color rgba="0 1 0 1"/>
       </material>
     </visual>
@@ -143,5 +143,5 @@
       <origin xyz="0.15 0 0" rpy="0 0 0"/>
       <geometry>
-        <box size="0.30 0.04 0.08"/>
+        <box size="1.2 0.04 0.08"/>
       </geometry>
       <material name="yellow">
@@ -158,5 +158,5 @@
       <origin xyz="0.15 0 0" rpy="0 0 0"/>
       <geometry>
-        <box size="0.30 0.04 0.08"/>
+        <box size="1.2 0.04 0.08"/>
       </geometry>
       <material name="yellow">
@@ -205,5 +205,5 @@
     <child link="left_finger"/>
     <axis xyz="0 1 0"/>
-    <limit effort="20" velocity="0.2" lower="0.0" upper="0.12"/>
+    <limit effort="20" velocity="0.2" lower="0.0" upper="0.4"/>
   </joint>
   <joint name="gripper_right" type="prismatic">
@@ -212,5 +212,5 @@
     <child link="right_finger"/>
     <axis xyz="0 -1 0"/>
-    <limit effort="20" velocity="0.2" lower="0.0" upper="0.12"/>
+    <limit effort="20" velocity="0.2" lower="0.0" upper="0.4"/>
   </joint>
   <link name="lidar_link"/>

Commit message: Added Gripper Publisher Features

File: install/TeleARM/share/TeleARM/urdf/telearm.urdf.xacro (robot description, xacro)
@@ -237,4 +237,20 @@
         <param name="min">-1</param>
         <param name="max">1</param>
+      </command_interface>
+      <state_interface name="position"/>
+      <state_interface name="velocity"/>
+    </joint>
+    <joint name="gripper_left">
+      <command_interface name="position">
+        <param name="min">0.0</param>
+        <param name="max">0.4</param>
+      </command_interface>
+      <state_interface name="position"/>
+      <state_interface name="velocity"/>
+    </joint>
+    <joint name="gripper_right">
+      <command_interface name="position">
+        <param name="min">0.0</param>
+        <param name="max">0.4</param>
       </command_interface>
       <state_interface name="position"/>

Commit message: Changed some stuff up

File: install/TeleARM/share/TeleARM/urdf/telearm.urdf.xacro (robot description, xacro)
@@ -1,353 +1 @@
-<?xml version="1.0"?>
-<robot name="robot" xmlns:xacro="http://ros.org/wiki/xacro">
-   <link name="body">
-    <inertial>
-      <mass value="1"/>
-      <inertia ixx=".1" ixy="0" ixz="0" iyy=".1" iyz="0" izz=".1" />
-    </inertial>
-    <visual>
-      <origin xyz="0 0 0" rpy="0 0 0" />
-      <geometry>
-        <mesh filename="file://$(find TeleARM)/meshes/body.STL" scale="1 1 1"/>
-      </geometry>
-      <material name="red">
-        <color rgba="1 0 0 1"/> <!-- Black color -->
-      </material>
-    </visual>
-  </link>
-  <link name="window">
-    <inertial>
-      <mass value="1"/>
-      <inertia ixx=".1" ixy="0" ixz="0" iyy=".1" iyz="0" izz=".1" />
-    </inertial>
-    <visual>
-      <origin xyz="0 0 0" rpy="0 0 0" />
-      <geometry>
-        <mesh filename="file://$(find TeleARM)/meshes/window.STL" scale="1 1 1"/>
-      </geometry>
-      <material name="red">
-        <color rgba="1 0 0 1"/> <!-- Black color -->
-      </material>
-    </visual>
-  </link>
-  <!-- Front Left -->
-  <link name="front_left_wheel">
-    <inertial>
-      <mass value="1"/>
-      <inertia ixx=".1" ixy="0" ixz="0" iyy=".1" iyz="0" izz=".1" />
-    </inertial>
-    <collision>
-      <origin xyz="0 0 0.16" rpy="0 0 0"/>
-      <geometry>
-        <cylinder radius="0.4175" length=".16"/>
-      </geometry>
-    </collision>
-    <visual>
-      <origin xyz="0 0 0" rpy="0 0 0" />
-      <geometry>
-        <mesh filename="file://$(find TeleARM)/meshes/wheel.STL" scale="1 1 1"/>
-      </geometry>
-      <material name="black">
-        <color rgba="0 0 0 1"/> <!-- Black color -->
-      </material>
-    </visual>
-  </link>
-  <!-- Front Right -->
-  <link name="front_right_wheel">
-    <inertial>
-      <mass value="1"/>
-      <inertia ixx=".1" ixy="0" ixz="0" iyy=".1" iyz="0" izz=".1" />
-    </inertial>
-    <collision>
-      <origin xyz="0 0 0.16" rpy="0 0 0"/>
-      <geometry>
-        <cylinder radius="0.4175" length=".16"/>
-      </geometry>
-    </collision>
-    <visual>
-      <origin xyz="0 0 0" rpy="0 0 0" />
-      <geometry>
-        <mesh filename="file://$(find TeleARM)/meshes/wheel.STL" scale="1 1 1"/>
-      </geometry>
-      <material name="black">
-        <color rgba="0 0 0 1"/> <!-- Black color -->
-      </material>
-    </visual>
-  </link>
-  <!-- Back Left -->
-  <link name="back_left_wheel">
-    <inertial>
-      <mass value="1"/>
-      <inertia ixx=".1" ixy="0" ixz="0" iyy=".1" iyz="0" izz=".1" />
-    </inertial>
-    <collision>
-      <origin xyz="0 0 0.16" rpy="0 0 0"/>
-      <geometry>
-        <cylinder radius="0.4175" length=".16"/>
-      </geometry>
-    </collision>
-    <visual>
-      <origin xyz="0 0 0" rpy="0 0 0" />
-      <geometry>
-        <mesh filename="file://$(find TeleARM)/meshes/wheel.STL" scale="1 1 1"/>
-      </geometry>
-      <material name="black">
-        <color rgba="0 0 0 1"/> <!-- Black color -->
-      </material>
-    </visual>
-  </link>
-  <!-- Back Right -->
-  <link name="back_right_wheel">
-    <inertial>
-      <mass value="1"/>
-      <inertia ixx=".1" ixy="0" ixz="0" iyy=".1" iyz="0" izz=".1" />
-    </inertial>
-    <collision>
-      <origin xyz="0 0 0.16" rpy="0 0 0"/>
-      <geometry>
-        <cylinder radius="0.4175" length=".16"/>
-      </geometry>
-    </collision>
-    <visual>
-      <origin xyz="0 0 0" rpy="0 0 0" />
-      <geometry>
-        <mesh filename="file://$(find TeleARM)/meshes/wheel.STL" scale="1 1 1"/>
-      </geometry>
-      <material name="black">
-        <color rgba="0 0 0 1"/> <!-- Black color -->
-      </material>
-    </visual>
-  </link>
-  <!-- Simple underbody gripper: base + 2 fingers -->
-  <link name="gripper_base">
-    <inertial>
-      <mass value="0.3"/>
-      <inertia ixx="0.01" ixy="0" ixz="0" iyy="0.01" iyz="0" izz="0.01"/>
-    </inertial>
-    <visual>
-      <origin xyz="0 0 0" rpy="0 0 0"/>
-      <geometry>
-        <box size="0.5 1.0 0.05"/>
-      </geometry>
-      <material name="green">
-        <color rgba="0 1 0 1"/>
-      </material>
-    </visual>
-  </link>
-  <link name="left_finger">
-    <inertial>
-      <mass value="0.1"/>
-      <inertia ixx="0.001" ixy="0" ixz="0" iyy="0.001" iyz="0" izz="0.001"/>
-    </inertial>
-    <visual>
-      <origin xyz="0.15 0 0" rpy="0 0 0"/>
-      <geometry>
-        <box size="1.2 0.04 0.08"/>
-      </geometry>
-      <material name="yellow">
-        <color rgba="1 0.85 0 1"/>
-      </material>
-    </visual>
-  </link>
-  <link name="right_finger">
-    <inertial>
-      <mass value="0.1"/>
-      <inertia ixx="0.001" ixy="0" ixz="0" iyy="0.001" iyz="0" izz="0.001"/>
-    </inertial>
-    <visual>
-      <origin xyz="0.15 0 0" rpy="0 0 0"/>
-      <geometry>
-        <box size="1.2 0.04 0.08"/>
-      </geometry>
-      <material name="yellow">
-        <color rgba="1 0.85 0 1"/>
-      </material>
-    </visual>
-  </link>
-  <joint name="body_to_window" type="fixed">
-    <origin xyz="0 0 0"/>
-    <parent link="body"/>
-    <child link="window"/>
-  </joint>
-  <joint name="body_to_front_left_wheel" type="continuous">
-    <origin xyz="1.505428 0.573211 0.055848" rpy="${-pi/2} 0 0"/>
-    <parent link="body"/>
-    <child link="front_left_wheel"/>
-    <axis xyz="0 0 1"/>
-  </joint>
-  <joint name="body_to_front_right_wheel" type="continuous">
-    <origin xyz="1.505428 -0.573211 0.055848" rpy="${pi/2} 0 0"/>
-    <parent link="body"/>
-    <child link="front_right_wheel"/>
-    <axis xyz="0 0 -1"/>
-  </joint>
-  <joint name="body_to_back_left_wheel" type="continuous">
-    <origin xyz="-1.505428 0.573211 0.055848" rpy="${-pi/2} 0 0"/>
-    <parent link="body"/>
-    <child link="back_left_wheel"/>
-    <axis xyz="0 0 1"/>
-  </joint>
-  <joint name="body_to_back_right_wheel" type="continuous">
-    <origin xyz="-1.505428 -0.573211 0.055848" rpy="${pi/2} 0 0"/>
-    <parent link="body"/>
-    <child link="back_right_wheel"/>
-    <axis xyz="0 0 -1"/>
-  </joint>
-  <!-- Gripper mounts under the front; slide fingers on Y to open/close -->
-  <joint name="body_to_gripper_base" type="fixed">
-    <origin xyz="2.4 0 0.15" rpy="0 0 0"/>
-    <parent link="body"/>
-    <child link="gripper_base"/>
-  </joint>
-  <joint name="gripper_left" type="prismatic">
-    <origin xyz="0 0.08 0" rpy="0 0 0"/>
-    <parent link="gripper_base"/>
-    <child link="left_finger"/>
-    <axis xyz="0 1 0"/>
-    <limit effort="20" velocity="0.2" lower="0.0" upper="0.4"/>
-  </joint>
-  <joint name="gripper_right" type="prismatic">
-    <origin xyz="0 -0.08 0" rpy="0 0 0"/>
-    <parent link="gripper_base"/>
-    <child link="right_finger"/>
-    <axis xyz="0 -1 0"/>
-    <limit effort="20" velocity="0.2" lower="0.0" upper="0.4"/>
-  </joint>
-  <link name="camera_link"/>
-  <joint name="body_to_camera_link" type="fixed">
-    <!-- Lower + pitched down so ~0.55 m floor boxes fill the image -->
-    <origin xyz="2.15 0 0.45" rpy="0 -0.55 0"/>
-    <parent link="body"/>
-    <child link="camera_link"/>
-  </joint>
-  <!-- Keep a lidar for /scan (avoidance). Camera is Image-only. -->
-  <link name="lidar_link"/>
-  <joint name="body_to_lidar_link" type="fixed">
-    <origin xyz="2.1 0 0.7" rpy="0 0 0"/>
-    <parent link="body"/>
-    <child link="lidar_link"/>
-  </joint>
-  <ros2_control name="GazeboSystem" type="system">
-    <hardware>
-      <plugin>gazebo_ros2_control/GazeboSystem</plugin>
-    </hardware>
-    <joint name="body_to_back_left_wheel">
-      <command_interface name="velocity">
-        <param name="min">-1</param>
-        <param name="max">1</param>
-      </command_interface>
-      <state_interface name="position"/>
-      <state_interface name="velocity"/>
-    </joint>
-    <joint name="body_to_back_right_wheel">
-      <command_interface name="velocity">
-        <param name="min">-1</param>
-        <param name="max">1</param>
-      </command_interface>
-      <state_interface name="position"/>
-      <state_interface name="velocity"/>
-    </joint>
-    <joint name="gripper_left">
-      <command_interface name="position">
-        <param name="min">0.0</param>
-        <param name="max">0.4</param>
-      </command_interface>
-      <state_interface name="position"/>
-      <state_interface name="velocity"/>
-    </joint>
-    <joint name="gripper_right">
-      <command_interface name="position">
-        <param name="min">0.0</param>
-        <param name="max">0.4</param>
-      </command_interface>
-      <state_interface name="position"/>
-      <state_interface name="velocity"/>
-    </joint>
-  </ros2_control>
-  <gazebo>
-    <!-- Joint state publisher -->
-    <plugin filename="libgazebo_ros2_control.so" name="gazebo_ros2_control">
-      <parameters>$(find TeleARM)/config/diff_drive_controller.yaml</parameters>
-    </plugin>
-  </gazebo>
-  <gazebo reference="body">
-    <material>Gazebo/Red</material>
-  </gazebo>
-  <gazebo reference="window">
-    <material>Gazebo/Black</material>
-  </gazebo>
-  <gazebo reference="front_left_wheel">
-    <material>Gazebo/Black</material>
-    <mu1 value="0.0"/>
-    <mu2 value="0.0"/>
-  </gazebo>
-  <gazebo reference="front_right_wheel">
-    <material>Gazebo/Black</material>
-    <mu1 value="0.0"/>
-    <mu2 value="0.0"/>
-  </gazebo>
-  <gazebo reference="back_left_wheel">
-    <material>Gazebo/Black</material>
-  </gazebo>
-  <gazebo reference="back_right_wheel">
-    <material>Gazebo/Black</material>
-  </gazebo>
-  <gazebo reference="camera_link">
-    <!-- RGB camera: publishes Image, NOT LaserScan.
-         Note: may crash Gazebo Classic on WSL (needs graphics Scene). -->
-    <sensor type="camera" name="rgb_camera">
-      <pose>0 0 0 0 0 0</pose>
-      <visualize>false</visualize>
-      <update_rate>10</update_rate>
-      <camera>
-        <horizontal_fov>1.3962634</horizontal_fov>
-        <image>
-          <width>320</width>
-          <height>240</height>
-          <format>R8G8B8</format>
-        </image>
-        <clip>
-          <near>0.1</near>
-          <far>20.0</far>
-        </clip>
-      </camera>
-      <plugin name="rgb_camera_controller" filename="libgazebo_ros_camera.so">
-        <ros>
-          <remapping>rgb_camera/image_raw:=/camera/image_raw</remapping>
-          <remapping>rgb_camera/camera_info:=/camera/camera_info</remapping>
-        </ros>
-        <camera_name>rgb_camera</camera_name>
-        <frame_name>camera_link</frame_name>
-      </plugin>
-    </sensor>
-  </gazebo>
-  <gazebo reference="lidar_link">
-    <sensor type="ray" name="lidar_sensor">
-      <pose>0 0 0 0 0 0</pose>
-      <visualize>false</visualize>
-      <update_rate>10</update_rate>
-      <ray>
-        <scan>
-          <horizontal>
-            <samples>720</samples>
-            <resolution>1</resolution>
-            <min_angle>-3.14159</min_angle>
-            <max_angle>3.14159</max_angle>
-          </horizontal>
-        </scan>
-        <range>
-          <min>0.12</min>
-          <max>12.0</max>
-          <resolution>0.01</resolution>
-        </range>
-      </ray>
-      <plugin name="lidar" filename="libgazebo_ros_ray_sensor.so">
-        <output_type>sensor_msgs/LaserScan</output_type>
-        <frame_name>lidar_link</frame_name>
-        <ros>
-          <remapping>~/out:=scan</remapping>
-        </ros>
-      </plugin>
-    </sensor>
-  </gazebo>
-</robot>
+/home/auric/ros2_ws/TeleARM/urdf/telearm.urdf.xacro

File: urdf/telearm.urdf.xacro (robot description, xacro)
@@ -134,4 +134,10 @@
       </material>
     </visual>
+    <collision>
+      <origin xyz="0 0 0" rpy="0 0 0"/>
+      <geometry>
+        <box size="0.5 1.0 0.05"/>
+      </geometry>
+    </collision>
   </link>
   <link name="left_finger">
@@ -141,7 +147,7 @@
     </inertial>
     <visual>
-      <origin xyz="0.15 0 0" rpy="0 0 0"/>
-      <geometry>
-        <box size="1.2 0.04 0.08"/>
+      <origin xyz="0.35 0 0" rpy="0 0 0"/>
+      <geometry>
+        <box size="1.0 0.06 0.10"/>
       </geometry>
       <material name="yellow">
@@ -149,4 +155,10 @@
       </material>
     </visual>
+    <collision>
+      <origin xyz="0.35 0 0" rpy="0 0 0"/>
+      <geometry>
+        <box size="1.0 0.06 0.10"/>
+      </geometry>
+    </collision>
   </link>
   <link name="right_finger">
@@ -156,7 +168,7 @@
     </inertial>
     <visual>
-      <origin xyz="0.15 0 0" rpy="0 0 0"/>
-      <geometry>
-        <box size="1.2 0.04 0.08"/>
+      <origin xyz="0.35 0 0" rpy="0 0 0"/>
+      <geometry>
+        <box size="1.0 0.06 0.10"/>
       </geometry>
       <material name="yellow">
@@ -164,4 +176,10 @@
       </material>
     </visual>
+    <collision>
+      <origin xyz="0.35 0 0" rpy="0 0 0"/>
+      <geometry>
+        <box size="1.0 0.06 0.10"/>
+      </geometry>
+    </collision>
   </link>
   <joint name="body_to_window" type="fixed">
@@ -194,7 +212,7 @@
     <axis xyz="0 0 -1"/>
   </joint>
-  <!-- Gripper mounts under the front; slide fingers on Y to open/close -->
+  <!-- Gripper under nose — keep clear of ground to avoid spawn yeet -->
   <joint name="body_to_gripper_base" type="fixed">
-    <origin xyz="2.4 0 0.15" rpy="0 0 0"/>
+    <origin xyz="2.35 0 0.22" rpy="0 0 0"/>
     <parent link="body"/>
     <child link="gripper_base"/>
