Commit message: Add camera link and update lidar joint settings
Added camera link and joint for camera integration. Updated lidar joint origin and modified visualization settings.

File: urdf/telearm.urdf.xacro (robot description, xacro)
@@ -214,8 +214,15 @@
     <limit effort="20" velocity="0.2" lower="0.0" upper="0.4"/>
   </joint>
+  <link name="camera_link"/>
+  <joint name="body_to_camera_link" type="fixed">
+    <!-- Lower + pitched down so ~0.55 m floor boxes fill the image -->
+    <origin xyz="2.15 0 0.45" rpy="0 -0.55 0"/>
+    <parent link="body"/>
+    <child link="camera_link"/>
+  </joint>
+  <!-- Keep a lidar for /scan (avoidance). Camera is Image-only. -->
   <link name="lidar_link"/>
   <joint name="body_to_lidar_link" type="fixed">
-    <!-- Front license-plate area (body mesh: x front~2.19, z roof~1.18, z bottom~0) -->
-    <origin xyz="2.1 0 0.9" rpy="0 0 0"/>
+    <origin xyz="2.1 0 0.7" rpy="0 0 0"/>
     <parent link="body"/>
     <child link="lidar_link"/>
@@ -286,8 +293,37 @@
     <material>Gazebo/Black</material>
   </gazebo>
+  <gazebo reference="camera_link">
+    <!-- RGB camera: publishes Image, NOT LaserScan.
+         Note: may crash Gazebo Classic on WSL (needs graphics Scene). -->
+    <sensor type="camera" name="rgb_camera">
+      <pose>0 0 0 0 0 0</pose>
+      <visualize>false</visualize>
+      <update_rate>10</update_rate>
+      <camera>
+        <horizontal_fov>1.3962634</horizontal_fov>
+        <image>
+          <width>320</width>
+          <height>240</height>
+          <format>R8G8B8</format>
+        </image>
+        <clip>
+          <near>0.1</near>
+          <far>20.0</far>
+        </clip>
+      </camera>
+      <plugin name="rgb_camera_controller" filename="libgazebo_ros_camera.so">
+        <ros>
+          <remapping>rgb_camera/image_raw:=/camera/image_raw</remapping>
+          <remapping>rgb_camera/camera_info:=/camera/camera_info</remapping>
+        </ros>
+        <camera_name>rgb_camera</camera_name>
+        <frame_name>camera_link</frame_name>
+      </plugin>
+    </sensor>
+  </gazebo>
   <gazebo reference="lidar_link">
     <sensor type="ray" name="lidar_sensor">
       <pose>0 0 0 0 0 0</pose>
-      <visualize>true</visualize>
+      <visualize>false</visualize>
       <update_rate>10</update_rate>
       <ray>

Commit message: Finally Done

File: urdf/telearm.urdf.xacro (robot description, xacro)
@@ -1,5 +1,24 @@
 <?xml version="1.0"?>
 <robot name="robot" xmlns:xacro="http://ros.org/wiki/xacro">
+  <!-- Overall forklift scale (meshes, wheels, nose). Gripper Z stays at box height. -->
+  <xacro:property name="S" value="1.35"/>
+  <xacro:property name="WR" value="${0.4175 * S}"/>
    <link name="body">
+    <inertial>
+      <!-- Heavy enough not to yeet; light enough to accelerate -->
+      <mass value="90"/>
+      <inertia ixx="35" ixy="0" ixz="0" iyy="70" iyz="0" izz="80" />
+    </inertial>
+    <visual>
+      <origin xyz="0 0 0" rpy="0 0 0" />
+      <geometry>
+        <mesh filename="file://$(find TeleARM)/meshes/body.STL" scale="${S} ${S} ${S}"/>
+      </geometry>
+      <material name="red">
+        <color rgba="1 0 0 1"/> <!-- Black color -->
+      </material>
+    </visual>
+  </link>
+  <link name="window">
     <inertial>
       <mass value="1"/>
@@ -9,5 +28,5 @@
       <origin xyz="0 0 0" rpy="0 0 0" />
       <geometry>
-        <mesh filename="file://$(find TeleARM)/meshes/body.STL" scale="1 1 1"/>
+        <mesh filename="file://$(find TeleARM)/meshes/window.STL" scale="${S} ${S} ${S}"/>
       </geometry>
       <material name="red">
@@ -16,35 +35,20 @@
     </visual>
   </link>
-  <link name="window">
-    <inertial>
-      <mass value="1"/>
-      <inertia ixx=".1" ixy="0" ixz="0" iyy=".1" iyz="0" izz=".1" />
-    </inertial>
-    <visual>
-      <origin xyz="0 0 0" rpy="0 0 0" />
-      <geometry>
-        <mesh filename="file://$(find TeleARM)/meshes/window.STL" scale="1 1 1"/>
-      </geometry>
-      <material name="red">
-        <color rgba="1 0 0 1"/> <!-- Black color -->
-      </material>
-    </visual>
-  </link>
   <!-- Front Left -->
   <link name="front_left_wheel">
     <inertial>
-      <mass value="1"/>
-      <inertia ixx=".1" ixy="0" ixz="0" iyy=".1" iyz="0" izz=".1" />
-    </inertial>
-    <collision>
-      <origin xyz="0 0 0.16" rpy="0 0 0"/>
-      <geometry>
-        <cylinder radius="0.4175" length=".16"/>
-      </geometry>
-    </collision>
-    <visual>
-      <origin xyz="0 0 0" rpy="0 0 0" />
-      <geometry>
-        <mesh filename="file://$(find TeleARM)/meshes/wheel.STL" scale="1 1 1"/>
+      <mass value="10"/>
+      <inertia ixx="0.6" ixy="0" ixz="0" iyy="0.6" iyz="0" izz="1.0" />
+    </inertial>
+    <collision>
+      <origin xyz="0 0 ${0.16 * S}" rpy="0 0 0"/>
+      <geometry>
+        <cylinder radius="${WR}" length="${0.16 * S}"/>
+      </geometry>
+    </collision>
+    <visual>
+      <origin xyz="0 0 0" rpy="0 0 0" />
+      <geometry>
+        <mesh filename="file://$(find TeleARM)/meshes/wheel.STL" scale="${S} ${S} ${S}"/>
       </geometry>
       <material name="black">
@@ -56,17 +60,17 @@
   <link name="front_right_wheel">
     <inertial>
-      <mass value="1"/>
-      <inertia ixx=".1" ixy="0" ixz="0" iyy=".1" iyz="0" izz=".1" />
-    </inertial>
-    <collision>
-      <origin xyz="0 0 0.16" rpy="0 0 0"/>
-      <geometry>
-        <cylinder radius="0.4175" length=".16"/>
-      </geometry>
-    </collision>
-    <visual>
-      <origin xyz="0 0 0" rpy="0 0 0" />
-      <geometry>
-        <mesh filename="file://$(find TeleARM)/meshes/wheel.STL" scale="1 1 1"/>
+      <mass value="10"/>
+      <inertia ixx="0.6" ixy="0" ixz="0" iyy="0.6" iyz="0" izz="1.0" />
+    </inertial>
+    <collision>
+      <origin xyz="0 0 ${0.16 * S}" rpy="0 0 0"/>
+      <geometry>
+        <cylinder radius="${WR}" length="${0.16 * S}"/>
+      </geometry>
+    </collision>
+    <visual>
+      <origin xyz="0 0 0" rpy="0 0 0" />
+      <geometry>
+        <mesh filename="file://$(find TeleARM)/meshes/wheel.STL" scale="${S} ${S} ${S}"/>
       </geometry>
       <material name="black">
@@ -78,17 +82,17 @@
   <link name="back_left_wheel">
     <inertial>
-      <mass value="1"/>
-      <inertia ixx=".1" ixy="0" ixz="0" iyy=".1" iyz="0" izz=".1" />
-    </inertial>
-    <collision>
-      <origin xyz="0 0 0.16" rpy="0 0 0"/>
-      <geometry>
-        <cylinder radius="0.4175" length=".16"/>
-      </geometry>
-    </collision>
-    <visual>
-      <origin xyz="0 0 0" rpy="0 0 0" />
-      <geometry>
-        <mesh filename="file://$(find TeleARM)/meshes/wheel.STL" scale="1 1 1"/>
+      <mass value="10"/>
+      <inertia ixx="0.6" ixy="0" ixz="0" iyy="0.6" iyz="0" izz="1.0" />
+    </inertial>
+    <collision>
+      <origin xyz="0 0 ${0.16 * S}" rpy="0 0 0"/>
+      <geometry>
+        <cylinder radius="${WR}" length="${0.16 * S}"/>
+      </geometry>
+    </collision>
+    <visual>
+      <origin xyz="0 0 0" rpy="0 0 0" />
+      <geometry>
+        <mesh filename="file://$(find TeleARM)/meshes/wheel.STL" scale="${S} ${S} ${S}"/>
       </geometry>
       <material name="black">
@@ -100,17 +104,17 @@
   <link name="back_right_wheel">
     <inertial>
-      <mass value="1"/>
-      <inertia ixx=".1" ixy="0" ixz="0" iyy=".1" iyz="0" izz=".1" />
-    </inertial>
-    <collision>
-      <origin xyz="0 0 0.16" rpy="0 0 0"/>
-      <geometry>
-        <cylinder radius="0.4175" length=".16"/>
-      </geometry>
-    </collision>
-    <visual>
-      <origin xyz="0 0 0" rpy="0 0 0" />
-      <geometry>
-        <mesh filename="file://$(find TeleARM)/meshes/wheel.STL" scale="1 1 1"/>
+      <mass value="10"/>
+      <inertia ixx="0.6" ixy="0" ixz="0" iyy="0.6" iyz="0" izz="1.0" />
+    </inertial>
+    <collision>
+      <origin xyz="0 0 ${0.16 * S}" rpy="0 0 0"/>
+      <geometry>
+        <cylinder radius="${WR}" length="${0.16 * S}"/>
+      </geometry>
+    </collision>
+    <visual>
+      <origin xyz="0 0 0" rpy="0 0 0" />
+      <geometry>
+        <mesh filename="file://$(find TeleARM)/meshes/wheel.STL" scale="${S} ${S} ${S}"/>
       </geometry>
       <material name="black">
@@ -119,14 +123,14 @@
     </visual>
   </link>
-  <!-- Simple underbody gripper: base + 2 fingers -->
+  <!-- Chunkier claw — open/close travel is obvious -->
   <link name="gripper_base">
     <inertial>
-      <mass value="0.3"/>
-      <inertia ixx="0.01" ixy="0" ixz="0" iyy="0.01" iyz="0" izz="0.01"/>
+      <mass value="0.5"/>
+      <inertia ixx="0.02" ixy="0" ixz="0" iyy="0.02" iyz="0" izz="0.02"/>
     </inertial>
     <visual>
       <origin xyz="0 0 0" rpy="0 0 0"/>
       <geometry>
-        <box size="0.5 1.0 0.05"/>
+        <box size="0.7 1.8 0.08"/>
       </geometry>
       <material name="green">
@@ -134,20 +138,15 @@
       </material>
     </visual>
-    <collision>
-      <origin xyz="0 0 0" rpy="0 0 0"/>
-      <geometry>
-        <box size="0.5 1.0 0.05"/>
-      </geometry>
-    </collision>
+    <!-- no collision on base — only fingers touch boxes (avoids yeeting them) -->
   </link>
   <link name="left_finger">
     <inertial>
-      <mass value="0.1"/>
-      <inertia ixx="0.001" ixy="0" ixz="0" iyy="0.001" iyz="0" izz="0.001"/>
-    </inertial>
-    <visual>
-      <origin xyz="0.35 0 0" rpy="0 0 0"/>
-      <geometry>
-        <box size="1.0 0.06 0.10"/>
+      <mass value="0.2"/>
+      <inertia ixx="0.002" ixy="0" ixz="0" iyy="0.002" iyz="0" izz="0.002"/>
+    </inertial>
+    <visual>
+      <origin xyz="0.45 0 0" rpy="0 0 0"/>
+      <geometry>
+        <box size="1.4 0.14 0.40"/>
       </geometry>
       <material name="yellow">
@@ -156,7 +155,7 @@
     </visual>
     <collision>
-      <origin xyz="0.35 0 0" rpy="0 0 0"/>
-      <geometry>
-        <box size="1.0 0.06 0.10"/>
+      <origin xyz="0.45 0 0" rpy="0 0 0"/>
+      <geometry>
+        <box size="1.4 0.14 0.40"/>
       </geometry>
     </collision>
@@ -164,11 +163,11 @@
   <link name="right_finger">
     <inertial>
-      <mass value="0.1"/>
-      <inertia ixx="0.001" ixy="0" ixz="0" iyy="0.001" iyz="0" izz="0.001"/>
-    </inertial>
-    <visual>
-      <origin xyz="0.35 0 0" rpy="0 0 0"/>
-      <geometry>
-        <box size="1.0 0.06 0.10"/>
+      <mass value="0.2"/>
+      <inertia ixx="0.002" ixy="0" ixz="0" iyy="0.002" iyz="0" izz="0.002"/>
+    </inertial>
+    <visual>
+      <origin xyz="0.45 0 0" rpy="0 0 0"/>
+      <geometry>
+        <box size="1.4 0.14 0.40"/>
       </geometry>
       <material name="yellow">
@@ -177,7 +176,7 @@
     </visual>
     <collision>
-      <origin xyz="0.35 0 0" rpy="0 0 0"/>
-      <geometry>
-        <box size="1.0 0.06 0.10"/>
+      <origin xyz="0.45 0 0" rpy="0 0 0"/>
+      <geometry>
+        <box size="1.4 0.14 0.40"/>
       </geometry>
     </collision>
@@ -189,5 +188,5 @@
   </joint>
   <joint name="body_to_front_left_wheel" type="continuous">
-    <origin xyz="1.505428 0.573211 0.055848" rpy="${-pi/2} 0 0"/>
+    <origin xyz="${1.505428 * S} ${0.573211 * S} ${0.055848 * S}" rpy="${-pi/2} 0 0"/>
     <parent link="body"/>
     <child link="front_left_wheel"/>
@@ -195,5 +194,5 @@
   </joint>
   <joint name="body_to_front_right_wheel" type="continuous">
-    <origin xyz="1.505428 -0.573211 0.055848" rpy="${pi/2} 0 0"/>
+    <origin xyz="${1.505428 * S} ${-0.573211 * S} ${0.055848 * S}" rpy="${pi/2} 0 0"/>
     <parent link="body"/>
     <child link="front_right_wheel"/>
@@ -201,5 +200,5 @@
   </joint>
   <joint name="body_to_back_left_wheel" type="continuous">
-    <origin xyz="-1.505428 0.573211 0.055848" rpy="${-pi/2} 0 0"/>
+    <origin xyz="${-1.505428 * S} ${0.573211 * S} ${0.055848 * S}" rpy="${-pi/2} 0 0"/>
     <parent link="body"/>
     <child link="back_left_wheel"/>
@@ -207,33 +206,33 @@
   </joint>
   <joint name="body_to_back_right_wheel" type="continuous">
-    <origin xyz="-1.505428 -0.573211 0.055848" rpy="${pi/2} 0 0"/>
+    <origin xyz="${-1.505428 * S} ${-0.573211 * S} ${0.055848 * S}" rpy="${pi/2} 0 0"/>
     <parent link="body"/>
     <child link="back_right_wheel"/>
     <axis xyz="0 0 -1"/>
   </joint>
-  <!-- Gripper under nose — keep clear of ground to avoid spawn yeet -->
+  <!-- Nose farther out (scaled); Z matches ~0.90 m box centers -->
   <joint name="body_to_gripper_base" type="fixed">
-    <origin xyz="2.35 0 0.22" rpy="0 0 0"/>
+    <origin xyz="${2.35 * S} 0 0.45" rpy="0 0 0"/>
     <parent link="body"/>
     <child link="gripper_base"/>
   </joint>
   <joint name="gripper_left" type="prismatic">
-    <origin xyz="0 0.08 0" rpy="0 0 0"/>
+    <origin xyz="0 0.16 0" rpy="0 0 0"/>
     <parent link="gripper_base"/>
     <child link="left_finger"/>
     <axis xyz="0 1 0"/>
-    <limit effort="20" velocity="0.2" lower="0.0" upper="0.4"/>
+    <!-- wide open vs tight close so claw motion is obvious -->
+    <limit effort="120" velocity="0.5" lower="0.0" upper="0.80"/>
   </joint>
   <joint name="gripper_right" type="prismatic">
-    <origin xyz="0 -0.08 0" rpy="0 0 0"/>
+    <origin xyz="0 -0.16 0" rpy="0 0 0"/>
     <parent link="gripper_base"/>
     <child link="right_finger"/>
     <axis xyz="0 -1 0"/>
-    <limit effort="20" velocity="0.2" lower="0.0" upper="0.4"/>
+    <limit effort="120" velocity="0.5" lower="0.0" upper="0.80"/>
   </joint>
   <link name="camera_link"/>
   <joint name="body_to_camera_link" type="fixed">
-    <!-- Lower + pitched down so ~0.55 m floor boxes fill the image -->
-    <origin xyz="2.15 0 0.45" rpy="0 -0.55 0"/>
+    <origin xyz="${2.15 * S} 0 0.55" rpy="0 -0.55 0"/>
     <parent link="body"/>
     <child link="camera_link"/>
@@ -242,5 +241,5 @@
   <link name="lidar_link"/>
   <joint name="body_to_lidar_link" type="fixed">
-    <origin xyz="2.1 0 0.7" rpy="0 0 0"/>
+    <origin xyz="${2.1 * S} 0 ${0.7 * S}" rpy="0 0 0"/>
     <parent link="body"/>
     <child link="lidar_link"/>
@@ -269,5 +268,5 @@
       <command_interface name="position">
         <param name="min">0.0</param>
-        <param name="max">0.4</param>
+        <param name="max">0.80</param>
       </command_interface>
       <state_interface name="position"/>
@@ -277,5 +276,5 @@
       <command_interface name="position">
         <param name="min">0.0</param>
-        <param name="max">0.4</param>
+        <param name="max">0.80</param>
       </command_interface>
       <state_interface name="position"/>
@@ -291,23 +290,42 @@
   <gazebo reference="body">
     <material>Gazebo/Red</material>
+    <selfCollide>false</selfCollide>
   </gazebo>
   <gazebo reference="window">
     <material>Gazebo/Black</material>
   </gazebo>
+  <!-- Front wheels are undriven — zero friction so they don't drag the car -->
   <gazebo reference="front_left_wheel">
     <material>Gazebo/Black</material>
-    <mu1 value="0.0"/>
-    <mu2 value="0.0"/>
+    <mu1>0.0</mu1>
+    <mu2>0.0</mu2>
   </gazebo>
   <gazebo reference="front_right_wheel">
     <material>Gazebo/Black</material>
-    <mu1 value="0.0"/>
-    <mu2 value="0.0"/>
+    <mu1>0.0</mu1>
+    <mu2>0.0</mu2>
   </gazebo>
   <gazebo reference="back_left_wheel">
     <material>Gazebo/Black</material>
+    <mu1>1.2</mu1>
+    <mu2>1.2</mu2>
   </gazebo>
   <gazebo reference="back_right_wheel">
     <material>Gazebo/Black</material>
+    <mu1>1.2</mu1>
+    <mu2>1.2</mu2>
+  </gazebo>
+  <!-- Grip friction — keep kp moderate so boxes don't get yeeted -->
+  <gazebo reference="left_finger">
+    <mu1>2.5</mu1>
+    <mu2>2.5</mu2>
+    <kp>1e4</kp>
+    <kd>10.0</kd>
+  </gazebo>
+  <gazebo reference="right_finger">
+    <mu1>2.5</mu1>
+    <mu2>2.5</mu2>
+    <kp>1e4</kp>
+    <kd>10.0</kd>
   </gazebo>
   <gazebo reference="camera_link">
